File: ADSCP/ADSCP.kicad_sch (KiCad schematic)
At the start: 0 parts

Commit message: add schematics
Other:
- sheet Sidechain 1 - Summing & Rectifier renamed Sidechain
Changed lines of the file:
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@@
 	(rectangle
 		(start 25.4 148.59)
-		(end 170.18 185.42)
+		(end 91.44 185.42)
 		(stroke
 			(width 1)
@@
 	)
 	(sheet
-		(at 41.91 158.75)
+		(at 44.45 158.75)
 		(size 25.4 17.78)
 		(exclude_from_sim no)
@@
 			(color 0 0 0 0.0000)
 		)
-		(property "Sheetname" "Sidechain 1 - Summing & Rectifier"
-			(at 29.972 156.972 0)
+		(property "Sheetname" "Sidechain"
+			(at 48.514 156.718 0)
 			(effects
 				(font
@@
 		)
 		(property "Sheetfile" "sidechain1.kicad_sch"
-			(at 41.148 177.8 0)
+			(at 43.688 177.8 0)
 			(effects
 				(font
