File: ADSCP/ADSCP.kicad_sch (KiCad schematic)
At the start: 0 parts

Commit message: add schematics
Other:
- added sheet Other schematics (other.kicad_sch)
- note added: "Other schematics"
Changed lines of the file:
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@@
+	)
+	(rectangle
+		(start 217.17 93.98)
+		(end 276.86 130.81)
+		(stroke
+			(width 1)
+			(type solid)
+		)
+		(fill
+			(type none)
+		)
 	)
 	(rectangle
@@
 		(fill
 			(type none)
+		)
+	)
+	(text "Other schematics"
+		(exclude_from_sim no)
+		(at 243.078 89.662 0)
+		(effects
+			(font
+				(size 4 4)
+				(thickness 0.8)
+				(bold yes)
+			)
 		)
 	)
@@
 				)
 			)
+		)
+	)
+	(sheet
+		(at 231.14 104.14)
+		(size 30.48 17.78)
+		(exclude_from_sim no)
+		(in_bom yes)
+		(on_board yes)
+		(dnp no)
+		(stroke
+			(width 0.1524)
+			(type solid)
+		)
+		(fill
+			(color 0 0 0 0.0000)
+		)
+		(property "Sheetname" "Other schematics"
+			(at 232.918 102.616 0)
+			(effects
+				(font
+					(size 2 2)
+					(thickness 0.4)
+					(bold yes)
+				)
+				(justify left bottom)
+			)
+		)
+		(property "Sheetfile" "other.kicad_sch"
+			(at 231.14 122.5046 0)
+			(effects
+				(font
+					(size 1.27 1.27)
+				)
+				(justify left top)
+			)
+		)
+		(instances
+			(project "ADSCP"
+				(path "/132f4570-4169-4ecf-b1f3-d724b5ad1d4e"
+					(page "8")
+				)
+			)
