File: ADSCP/inputbuffer.kicad_sch (KiCad schematic)
At the start: 15 parts, among them J1 Input_Jack_L, J2 Input_Jack_R, U1 TL074 or OPA1644, U3 TL074 or OPA1644, U4 TL074

Commit message: add schematics
Parts:
- C1, C3: footprint Capacitor_THT:CP_Radial_D8.0mm_P3.50mm -> Capacitor_THT:C_Radial_D8.0mm_H7.0mm_P3.50mm
Changed lines of the file:
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@@
 			)
 		)
-		(property "Footprint" "Capacitor_THT:CP_Radial_D8.0mm_P3.50mm"
+		(property "Footprint" "Capacitor_THT:C_Radial_D8.0mm_H7.0mm_P3.50mm"
 			(at 162.2552 52.07 0)
 			(effects
@@
 			)
 		)
-		(property "Footprint" "Capacitor_THT:CP_Radial_D8.0mm_P3.50mm"
+		(property "Footprint" "Capacitor_THT:C_Radial_D8.0mm_H7.0mm_P3.50mm"
 			(at 86.0552 50.8 0)
 			(effects
