File: ADSCP/inputbuffer.kicad_sch (KiCad schematic)
At the start: 16 parts, among them J1 Input_Jack_L, J2 Input_Jack_R, U1 TL074 or OPA1644, U3 TL074 or OPA1644, U4 TL074, U5 TL072

Commit message: add schematics
Parts:
- removed unit 5 of U1
- removed unit 5 of U3
- removed U4: TL074, symbol Device:Opamp_Quad
- removed U5: TL072, symbol Device:Opamp_Dual
Connections:
- net Input Buffer L Out is gone; now on net BLEND_DRY_L: U1.1
- net Input Buffer R Out is gone; now on net BLEND_DRY_R: U3.1
- net BLEND_DRY_L: no longer R2.1
- net BLEND_DRY_R: no longer R5.1
- net TO_VCA_IN_L renamed VCA_IN_L
- net TO_VCA_IN_R renamed VCA_IN_R
- new net SIDECHAIN_L: R2.1
- new net SIDECHAIN_R: R5.1
Other:
- moved on the sheet: C1, C2, C3, C4, J1, J2, R1, R2, R3, R4, R5, R6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

Commit message: add pcb
Parts:
- U3: footprint (none) -> Package_DIP:DIP-14_W7.62mm
Changed lines of the file:
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@@
 			)
 		)
-		(property "Footprint" ""
+		(property "Footprint" "Package_DIP:DIP-14_W7.62mm"
 			(at 189.23 90.17 0)
 			(effects
