File: ADSCP/SSI2164.kicad_sch (KiCad schematic)
At the start: 5 parts, among them U2 SSI2164

Commit message: add schematics
Connections:
- net CV_IN renamed CV_IN_L
- net CV_IN_L: no longer U2.6 (VC2)
- new net CV_IN_R: U2.6 (VC2)
Changed lines of the file:
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@@
 		)
 	)
-	(global_label "CV_IN"
+	(global_label "CV_IN_L"
 		(shape input)
 		(at 105.41 71.12 180)
@@
 		)
 		(property "Intersheetrefs" "${INTERSHEET_REFS}"
-			(at 97.1633 71.12 0)
+			(at 95.1676 71.12 0)
 			(effects
 				(font
@@
 		)
 	)
-	(global_label "CV_IN"
+	(global_label "CV_IN_R"
 		(shape input)
 		(at 105.41 78.74 180)
@@
 		)
 		(property "Intersheetrefs" "${INTERSHEET_REFS}"
-			(at 97.1633 78.74 0)
+			(at 94.9257 78.74 0)
 			(effects
 				(font

Commit message: add schematics
Changed lines of the file:
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@@
 	(global_label "-15V"
 		(shape input)
-		(at 129.54 114.3 270)
-		(fields_autoplaced yes)
-		(effects
-			(font
-				(size 1.27 1.27)
-			)
-			(justify right)
-		)
-		(property "Intersheetrefs" "${INTERSHEET_REFS}"
-			(at 129.54 122.3652 90)
-			(effects
-				(font
-					(size 1.27 1.27)
-				)
-				(justify right)
+		(at 129.54 114.3 0)
+		(fields_autoplaced yes)
+		(effects
+			(font
+				(size 1.27 1.27)
+			)
+			(justify left)
+		)
+		(property "Intersheetrefs" "${INTERSHEET_REFS}"
+			(at 137.6052 114.3 0)
+			(effects
+				(font
+					(size 1.27 1.27)
+				)
+				(justify left)
 				(hide yes)
 			)
@@
 	(global_label "+15V"
 		(shape input)
-		(at 129.54 57.15 90)
+		(at 129.54 57.15 0)
 		(fields_autoplaced yes)
 		(effects
@@
 		)
 		(property "Intersheetrefs" "${INTERSHEET_REFS}"
-			(at 129.54 49.0848 90)
+			(at 137.6052 57.15 0)
 			(effects
 				(font
@@
 		(on_board yes)
 		(dnp no)
-		(fields_autoplaced yes)
 		(property "Reference" "C5"
-			(at 125.73 53.34 90)
+			(at 125.73 54.864 90)
 			(effects
 				(font
@@
 		)
 		(property "Value" "0.1uF"
-			(at 125.73 55.88 90)
-			(effects
-				(font
+			(at 125.73 57.404 90)
+			(effects
+				(font
