File: ADSCP/Grmeter.kicad_sch (KiCad schematic)
At the start: 13 parts, among them U5 TL072, U6 LM3914N

Commit message: add schematics
Other:
- moved on the sheet: C11, D10, D5, D6, D7, D8, D9, R32, Scale_Adjust_Trim, U6

Commit message: add pcb
Parts:
- U5: footprint (none) -> Package_DIP:DIP-8_W7.62mm
- renumbered Scale_Adjust_Trim to Scale_Adjust_Trim1
Changed lines of the file:
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@@
 		(on_board yes)
 		(dnp no)
-		(property "Reference" "Scale_Adjust_Trim"
+		(property "Reference" "Scale_Adjust_Trim1"
 			(at 143.002 110.744 90)
 			(effects
@@
 			(project "ADSCP"
 				(path "/132f4570-4169-4ecf-b1f3-d724b5ad1d4e/187ea13d-2cf3-4f61-b7ee-48a5d293ae6b"
-					(reference "Scale_Adjust_Trim")
+					(reference "Scale_Adjust_Trim1")
 					(unit 1)
 				)
@@
 			)
 		)
-		(property "Footprint" ""
+		(property "Footprint" "Package_DIP:DIP-8_W7.62mm"
 			(at 55.88 46.99 0)
 			(effects
@@
 			)
 		)
-		(property "Footprint" ""
+		(property "Footprint" "Package_DIP:DIP-8_W7.62mm"
 			(at 55.88 68.58 0)
 			(effects
