File: ADSCP/blend_and_output.kicad_sch (KiCad schematic)
At the start: 12 parts, among them J3 Output_Jack_L, J4 Output_Jack_R, U1 TL074 or OPA1644, U3 TL074 or OPA1644

Commit message: add schematics
Connections:
- net OUTPUT_JACK_R: now reaches J4.T, R20.2
- net OUTPUT_JACK_L: now reaches J3.T, R17.2
Other:
- moved on the sheet: Blend_L, Blend_R, J3, J4, R15, R16, R17, R18, R19, R20, U1D, U3D

Commit message: add pcb
Parts:
- U3: footprint (none) -> Package_DIP:DIP-14_W7.62mm
- renumbered Blend_L to Blend_L1, Blend_R to Blend_R1
Changed lines of the file:
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@@
 		(on_board yes)
 		(dnp no)
-		(property "Reference" "Blend_R"
+		(property "Reference" "Blend_R1"
 			(at 115.57 105.41 90)
 			(effects
@@
 			(project "ADSCP"
 				(path "/132f4570-4169-4ecf-b1f3-d724b5ad1d4e/47de73ca-0318-4417-b2e7-58ec17641450"
-					(reference "Blend_R")
+					(reference "Blend_R1")
 					(unit 1)
 				)
@@
 			)
 		)
-		(property "Footprint" ""
+		(property "Footprint" "Package_DIP:DIP-14_W7.62mm"
 			(at 146.05 107.95 0)
 			(effects
@@
 		(on_board yes)
 		(dnp no)
-		(property "Reference" "Blend_L"
+		(property "Reference" "Blend_L1"
 			(at 115.57 64.77 90)
 			(effects
@@
 			(project "ADSCP"
 				(path "/132f4570-4169-4ecf-b1f3-d724b5ad1d4e/47de73ca-0318-4417-b2e7-58ec17641450"
-					(reference "Blend_L")
+					(reference "Blend_L1")
 					(unit 1)
 				)
