File: ADSCP/ivc_mug.kicad_sch (KiCad schematic)
At the start: 12 parts, among them U1 TL074 or OPA1644, U3 TL074 or OPA1644

Commit message: add schematics
Connections:
- net IV_OUT_L: no longer names the net of C7.1, R10.2, R9.2, U1.7
- net IV_OUT_R: no longer names the net of C8.1, R12.2, R13.2, U3.7
Other:
- moved on the sheet: C7, C8, MakeUpGain_L, MakeUpGain_R, R10, R11, R12, R13, R14, R9, U1B, U1C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

Commit message: add pcb
Parts:
- U3: footprint (none) -> Package_DIP:DIP-14_W7.62mm
- renumbered MakeUpGain_L to MakeUpGain_L1, MakeUpGain_R to MakeUpGain_R1
Changed lines of the file:
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@@
 			)
 		)
-		(property "Footprint" ""
+		(property "Footprint" "Package_DIP:DIP-14_W7.62mm"
 			(at 166.37 81.28 0)
 			(effects
@@
 		(on_board yes)
 		(dnp no)
-		(property "Reference" "MakeUpGain_R"
+		(property "Reference" "MakeUpGain_R1"
 			(at 176.53 101.6 90)
 			(effects
@@
 			(project "ADSCP"
 				(path "/132f4570-4169-4ecf-b1f3-d724b5ad1d4e/9a0a4327-39a8-4e8b-913c-f35a475a8204"
-					(reference "MakeUpGain_R")
+					(reference "MakeUpGain_R1")
 					(unit 1)
 				)
@@
 			)
 		)
-		(property "Footprint" ""
+		(property "Footprint" "Package_DIP:DIP-14_W7.62mm"
 			(at 167.64 128.27 0)
 			(effects
@@
 		(on_board yes)
 		(dnp no)
-		(property "Reference" "MakeUpGain_L"
+		(property "Reference" "MakeUpGain_L1"
 			(at 111.76 101.6 90)
 			(effects
@@
 			(project ""
 				(path "/132f4570-4169-4ecf-b1f3-d724b5ad1d4e/9a0a4327-39a8-4e8b-913c-f35a475a8204"
-					(reference "MakeUpGain_L")
+					(reference "MakeUpGain_L1")
 					(unit 1)
 				)
