File: ADSCP/other.kicad_sch (KiCad schematic)
At the start: 26 parts, among them J5 +DD1718PA Module, J6 -DD1718PA Module, SW1 Deep_Punch_Switch, SW2 Deep_Punch_Switch, U1 TL074 or OPA1644, U3 TL074 or OPA1644, U4 TL074, U5 TL072

Commit message: add pcb
Parts:
- D11: footprint (none) -> LED_THT:LED_D3.0mm
- SW1: value Deep_Punch_Switch -> Diode Saturator Switch
- U3, U4: footprint (none) -> Package_DIP:DIP-14_W7.62mm
- U5: footprint (none) -> Package_DIP:DIP-8_W7.62mm
Changed lines of the file:
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@@
 			)
 		)
-		(property "Footprint" ""
+		(property "Footprint" "Package_DIP:DIP-14_W7.62mm"
 			(at 215.9 129.54 0)
 			(effects
@@
 			)
 		)
-		(property "Footprint" ""
+		(property "Footprint" "Package_DIP:DIP-14_W7.62mm"
 			(at 190.5 129.54 0)
 			(effects
@@
 			)
 		)
-		(property "Footprint" ""
+		(property "Footprint" "LED_THT:LED_D3.0mm"
 			(at 109.22 50.8 0)
 			(effects
@@
 			)
 		)
-		(property "Footprint" ""
+		(property "Footprint" "Package_DIP:DIP-8_W7.62mm"
 			(at 232.41 129.54 0)
 			(effects
@@
 			)
 		)
-		(property "Value" "Deep_Punch_Switch"
+		(property "Value" "Diode Saturator Switch"
 			(at 83.82 144.78 0)
 			(effects
