File: ADSCP/sidechain1.kicad_sch (KiCad schematic)
At the start: 7 parts, among them U4 TL074

Commit message: add schematics
Parts:
- added Attack_Pot: 50kA, Connector_PinHeader_2.54mm:PinHeader_1x03_P2.54mm_Vertical, symbol Device:R_Potentiometer
- added C9: 10uF, Capacitor_THT:CP_Radial_D8.0mm_P3.50mm, symbol Device:C_Polarized
- added CV_Trim_L, CV_Trim_R: 10k, Potentiometer_THT:Potentiometer_Runtron_RM-065_Vertical, symbol Device:R_Potentiometer_Trim
- added D3, D4: 1N4148, Diode_THT:D_DO-35_SOD27_P7.62mm_Horizontal, symbol Device:D
- added R25, R26, R27, R28, R30: 10k, Resistor_THT:R_Axial_DIN0207_L6.3mm_D2.5mm_P2.54mm_Vertical, symbol Device:R
- added R29: 470R, Resistor_THT:R_Axial_DIN0207_L6.3mm_D2.5mm_P2.54mm_Vertical, symbol Device:R
- added Release_Pot: 250kA, Connector_PinHeader_2.54mm:PinHeader_1x03_P2.54mm_Vertical, symbol Device:R_Potentiometer
- added Retio_Pot, Threshold_Pot: 50kB, Connector_PinHeader_2.54mm:PinHeader_1x03_P2.54mm_Vertical, symbol Device:R_Potentiometer
Connections:
- net GND: now also U4.12 (+), C9.2, R29.1, Threshold_Pot.3
- net RECTIFIED_DC: now also D1.1 (K), R25.2, R26.1; no longer D1.2 (A), D2.1 (K), U4.7
- net at U4.13 (-): now also R28.2, R30.1
- net at U4.14: now also CV_Trim_L.1, CV_Trim_R.1, R30.2
- net at D2.2 (A), R24.2, U4.6 (-): now also R25.1; no longer D1.1 (K)
- net at U4.10 (+): now also R26.2
- net at U4.8: now also D3.2 (A)
- net at U4.9 (-): now also R27.2, Retio_Pot.3
- new net: Attack_Pot.3, D4.1 (K)
- new net: D1.2 (A), D2.1 (K), U4.7
- new net: D3.1 (K), Retio_Pot.1
- new net: R27.1, Threshold_Pot.2
- new net: R29.2, Release_Pot.2
- new net +15V: Threshold_Pot.1
- new net CV_IN_L: CV_Trim_L.2
- new net CV_IN_R: CV_Trim_R.2
- new net Point_X: Attack_Pot.2, C9.1, D4.2 (A), R28.1, Release_Pot.3, Retio_Pot.2
- no-connect marks 0 -> 4
Other:
- note added: "SC-1 Summing & Rectifier"
- note added: "SC-2 Threshold & Ratio"
- note added: "SC-3 Stereo Link, Timing & CV Output"
- moved on the sheet: D1, D2, R21, R22, R23, R24, U4A, U4B, U4C, U4D

Commit message: add schematics
Other:
- moved on the sheet: CV_Trim_L, CV_Trim_R, D1, D2, D3, R21, R22, R23, R24, R25, R26, R27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

Commit message: add pcb
Parts:
- U4: footprint (none) -> Package_DIP:DIP-14_W7.62mm
- renumbered Attack_Pot to Attack_Pot1, CV_Trim_L to CV_Trim_L1, CV_Trim_R to CV_Trim_R1, Release_Pot to Release_Pot1, Retio_Pot to Retio_Pot1, Threshold_Pot to Threshold_Pot1
Changed lines of the file:
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@@
 		)
 	)
-	(global_label "SIDECHAIN_L"
+	(global_label "Point_X"
 		(shape input)
-		(at 36.83 44.45 180)
-		(fields_autoplaced yes)
-		(effects
-			(font
-				(size 1.27 1.27)
-			)
-			(justify right)
-		)
-		(property "Intersheetrefs" "${INTERSHEET_REFS}"
-			(at 21.9914 44.45 0)
-			(effects
-				(font
-					(size 1.27 1.27)
-				)
-				(justify right)
-				(hide yes)
-			)
-		)
-	)
-	(global_label "CV_IN_L"
-		(shape input)
-		(at 161.29 137.16 0)
+		(at 36.83 121.92 180)
 		(fields_autoplaced yes)
 		(effects
@@
 				(thickness 0.1588)
 			)
-			(justify left)
+			(justify right)
 		)
 		(property "Intersheetrefs" "${INTERSHEET_REFS}"
-			(at 171.5324 137.16 0)
-			(effects
-				(font
-					(size 1.27 1.27)
-				)
-				(justify left)
-				(hide yes)
-			)
-		)
-	)
-	(global_label "CV_IN_R"
+			(at 26.7692 121.92 0)
+			(effects
+				(font
+					(size 1.27 1.27)
+				)
+				(justify right)
+				(hide yes)
+			)
+		)
+	)
+	(global_label "SIDECHAIN_L"
 		(shape input)
-		(at 161.29 144.78 0)
+		(at 36.83 44.45 180)
+		(fields_autoplaced yes)
+		(effects
+			(font
+				(size 1.27 1.27)
+			)
+			(justify right)
+		)
+		(property "Intersheetrefs" "${INTERSHEET_REFS}"
+			(at 21.9914 44.45 0)
+			(effects
+				(font
+					(size 1.27 1.27)
+				)
+				(justify right)
+				(hide yes)
+			)
+		)
+	)
+	(global_label "CV_IN_L"
+		(shape input)
+		(at 161.29 137.16 0)
 		(fields_autoplaced yes)
 		(effects
@@
 		)
 		(property "Intersheetrefs" "${INTERSHEET_REFS}"
-			(at 171.7743 144.78 0)
+			(at 171.5324 137.16 0)
 			(effects
 				(font
@@
 		)
 	)
-	(global_label "SIDECHAIN_R"
+	(global_label "CV_IN_R"
 		(shape input)
-		(at 36.83 62.23 180)
-		(fields_autoplaced yes)
-		(effects
-			(font
-				(size 1.27 1.27)
-			)
-			(justify right)
-		)
-		(property "Intersheetrefs" "${INTERSHEET_REFS}"
-			(at 21.7495 62.23 0)
-			(effects
-				(font
-					(size 1.27 1.27)
-				)
-				(justify right)
-				(hide yes)
-			)
-		)
-	)
-	(global_label "RECTIFIED_DC"
-		(shape input)
-		(at 137.16 64.77 0)
+		(at 161.29 144.78 0)
 		(fields_autoplaced yes)
 		(effects
@@
 		)
 		(property "Intersheetrefs" "${INTERSHEET_REFS}"
-			(at 153.0266 64.77 0)
+			(at 171.7743 144.78 0)
 			(effects
 				(font
@@
 				)
 				(justify left)
+				(hide yes)
+			)
+		)
+	)
+	(global_label "SIDECHAIN_R"
+		(shape input)
+		(at 36.83 62.23 180)
+		(fields_autoplaced yes)
+		(effects
+			(font
+				(size 1.27 1.27)
+			)
+			(justify right)
+		)
+		(property "Intersheetrefs" "${INTERSHEET_REFS}"
+			(at 21.7495 62.23 0)
+			(effects
+				(font
+					(size 1.27 1.27)
+				)
+				(justify right)
 				(hide yes)
 			)
@@
 	(global_label "RECTIFIED_DC"
 		(shape input)
-		(at 200.66 44.45 180)
+		(at 137.16 64.77 0)
 		(fields_autoplaced yes)
 		(effects
@@
 				(thickness 0.1588)
 			)
-			(justify right)
+			(justify left)
 		)
 		(property "Intersheetrefs" "${INTERSHEET_REFS}"
-			(at 184.7934 44.45 0)
-			(effects
-				(font
-					(size 1.27 1.27)
-				)
-				(justify right)
-				(hide yes)
-			)
-		)
-	)
-	(global_label "ST_LINK_TIMING"
+			(at 153.0266 64.77 0)
+			(effects
+				(font
+					(size 1.27 1.27)
+				)
+				(justify left)
+				(hide yes)
+			)
+		)
+	)
+	(global_label "RECTIFIED_DC"
 		(shape input)
-		(at 36.83 121.92 180)
+		(at 200.66 44.45 180)
 		(fields_autoplaced yes)
 		(effects
@@
 		)
 		(property "Intersheetrefs" "${INTERSHEET_REFS}"
-			(at 19.27 121.92 0)
+			(at 184.7934 44.45 0)
 			(effects
 				(font
@@
 	(global_label "Point_X"
 		(shape input)
-		(at 68.58 129.54 90)
+		(at 105.41 139.7 180)
 		(fields_autoplaced yes)
 		(effects
@@
 				(thickness 0.1588)
 			)
-			(justify left)
+			(justify right)
 		)
 		(property "Intersheetrefs" "${INTERSHEET_REFS}"
-			(at 68.58 119.4792 90)
-			(effects
-				(font
-					(size 1.27 1.27)
-				)
-				(justify left)
+			(at 95.3492 139.7 0)
+			(effects
+				(font
+					(size 1.27 1.27)
+				)
+				(justify right)
 				(hide yes)
 			)
@@
 	(global_label "Point_X"
 		(shape input)
-		(at 105.41 139.7 180)
+		(at 234.95 54.61 180)
 		(fields_autoplaced yes)
 		(effects
@@
 		)
 		(property "Intersheetrefs" "${INTERSHEET_REFS}"
-			(at 95.3492 139.7 0)
+			(at 224.8892 54.61 0)
 			(effects
 				(font
@@
 		)
 	)
-	(global_label "ST_LINK_TIMING"
-		(shape input)
-		(at 234.95 54.61 180)
-		(fields_autoplaced yes)
-		(effects
-			(font
-				(size 1.27 1.27)
-				(thickness 0.1588)
-			)
-			(justify right)
-		)
-		(property "Intersheetrefs" "${INTERSHEET_REFS}"
-			(at 217.39 54.61 0)
-			(effects
-				(font
-					(size 1.27 1.27)
-				)
-				(justify right)
-				(hide yes)
-			)
-		)
-	)
 	(symbol
 		(lib_id "power:GND")
@@
 			)
 		)
-		(property "Footprint" ""
+		(property "Footprint" "Package_DIP:DIP-14_W7.62mm"
 			(at 127 137.16 0)
 			(effects
@@
 			)
 		)
-		(property "Footprint" ""
+		(property "Footprint" "Package_DIP:DIP-14_W7.62mm"
 			(at 81.28 67.31 0)
 			(effects
@@
 		(on_board yes)
 		(dnp no)
-		(property "Reference" "Attack_Pot"
+		(property "Reference" "Attack_Pot1"
 			(at 58.42 115.57 90)
 			(effects
@@
 			(project "ADSCP"
 				(path "/132f4570-4169-4ecf-b1f3-d724b5ad1d4e/0b4d4bfd-31c8-4c19-84f1-17153586bb4a"
-					(reference "Attack_Pot")
+					(reference "Attack_Pot1")
 					(unit 1)
 				)
@@
 		(on_board yes)
 		(dnp no)
-		(property "Reference" "CV_Trim_L"
+		(property "Reference" "CV_Trim_L1"
 			(at 151.13 127 90)
 			(effects
@@
 			(project ""
 				(path "/132f4570-4169-4ecf-b1f3-d724b5ad1d4e/0b4d4bfd-31c8-4c19-84f1-17153586bb4a"
-					(reference "CV_Trim_L")
+					(reference "CV_Trim_L1")
 					(unit 1)
 				)
@@
 			)
 		)
-		(property "Footprint" ""
+		(property "Footprint" "Package_DIP:DIP-14_W7.62mm"
 			(at 224.79 46.99 0)
 			(effects
@@
 		(on_board yes)
 		(dnp no)
-		(property "Reference" "Retio_Pot"
+		(property "Reference" "Retio_Pot1"
 			(at 240.284 57.15 90)
 			(effects
@@
 			(project "ADSCP"
 				(path "/132f4570-4169-4ecf-b1f3-d724b5ad1d4e/0b4d4bfd-31c8-4c19-84f1-17153586bb4a"
-					(reference "Retio_Pot")
+					(reference "Retio_Pot1")
 					(unit 1)
 				)
@@
 			)
 		)
-		(property "Footprint" ""
+		(property "Footprint" "Package_DIP:DIP-14_W7.62mm"
 			(at 114.3 64.77 0)
 			(effects
@@
 		(on_board yes)
 		(dnp no)
-		(property "Reference" "CV_Trim_R"
+		(property "Reference" "CV_Trim_R1"
 			(at 151.13 147.32 90)
 			(effects
@@
 			(project "ADSCP"
 				(path "/132f4570-4169-4ecf-b1f3-d724b5ad1d4e/0b4d4bfd-31c8-4c19-84f1-17153586bb4a"
-					(reference "CV_Trim_R")
+					(reference "CV_Trim_R1")
 					(unit 1)
 				)
@@
 		(on_board yes)
 		(dnp no)
-		(property "Reference" "Release_Pot"
+		(property "Reference" "Release_Pot1"
 			(at 72.39 132.08 90)
 			(effects
@@
 			(project "ADSCP"
 				(path "/132f4570-4169-4ecf-b1f3-d724b5ad1d4e/0b4d4bfd-31c8-4c19-84f1-17153586bb4a"
-					(reference "Release_Pot")
+					(reference "Release_Pot1")
 					(unit 1)
 				)
@@
 		(on_board yes)
 		(dnp no)
-		(property "Reference" "Threshold_Pot"
+		(property "Reference" "Threshold_Pot1"
 			(at 186.69 60.96 90)
 			(effects
@@
 			(project "ADSCP"
 				(path "/132f4570-4169-4ecf-b1f3-d724b5ad1d4e/0b4d4bfd-31c8-4c19-84f1-17153586bb4a"
-					(reference "Threshold_Pot")
+					(reference "Threshold_Pot1")
 					(unit 1)
 				)
